Commit message: Update allegro_hand_description_3f.urdf

File: src/allegro_hand_controllers/urdf/allegro_hand_description_3f.urdf (robot description, URDF)
Before this commit: robot allegro_hand, 14 links, 13 joints
Joints:
- joint joint_2_0: limit lower=-0.05 upper=1.45 effort=15 velocity=7 -> lower=-1.45 upper=1.45 effort=15 velocity=7
- joint joint_5_0: limit lower=-0.05 upper=1.45 effort=15 velocity=7 -> lower=-1.45 upper=1.45 effort=15 velocity=7
- joint joint_8_0: limit lower=-0.05 upper=1.45 effort=15 velocity=7 -> lower=-1.45 upper=1.45 effort=15 velocity=7

Commit message: Add files via upload
Change mass & inertia

File: src/allegro_hand_controllers/urdf/allegro_hand_description_3f.urdf (robot description, URDF)
Before this commit: robot allegro_hand, 14 links, 13 joints
Links:
- link link_0_0: mass 0.4154 -> 0.04374
- link link_1_0: mass 0.4154 -> 0.09852
- link link_2_0: mass 0.4154 -> 0.0687
- link link_2_0_tip: mass 0.4154 -> 0.001
- link link_3_0: mass 0.4154 -> 0.04374
- link link_4_0: mass 0.4154 -> 0.09852
- link link_5_0: mass 0.4154 -> 0.0687
- link link_5_0_tip: mass 0.4154 -> 0.001
- link link_6_0: mass 0.4154 -> 0.04374
- link link_7_0: mass 0.4154 -> 0.09852
- link link_8_0: mass 0.4154 -> 0.0687
- link link_8_0_tip: mass 0.4154 -> 0.001
